File: juno-chorus-clone.sch (KiCad schematic (older format))
At the start: 168 parts, among them P1 15VAC_IN, P2 AUDIO_IN, P3 AUDIO_OUT_1, P4 AUDIO_OUT_2, Q1 2SC1815, Q10 2SC1815, Q11 2SA1015, Q12 2SA1015, Q13 2SC1815, Q14 2SA1015, Q15 2SA1015, Q16 2SK30, Q17 2SK30, Q18 2SA1015, Q19 2SA1015, Q2 2SC1815, Q3 2SA1015, Q4 2SA1015, Q5 2SC1815, Q6 2SC1815, Q7 2SA1015, Q8 2SA1015, Q9 2SC1815, SW1 SW_PUSH, U1 TL082, U10 TL082, U2 LM7815CT, U3 LM7915CT, U4 TL082, U5 MN3009, U6 MN3101, U7 MN3009, U8 MN3101, U9 TL082

Commit message: Add paste layer and gerber files
Parts:
- C1, C12, C13, C14, C15, C17, C19, C2, C23, C3, C30, C31, C4: symbol CP1 -> juno-chorus-clone-rescue:CP1
- C10, C11, C16, C18, C20, C21, C24, C25, C26, C27, C28, C29, C32, C33, C34, C35, C5, C6, C7, C8, C9: symbol C -> juno-chorus-clone-rescue:C
- D1, D2: symbol DIODESCH -> juno-chorus-clone-rescue:DIODESCH
- D3, D4, D5, D6, D7: symbol DIODE -> juno-chorus-clone-rescue:DIODE
- P1, P2, P3, P4: symbol CONN_2 -> juno-chorus-clone-rescue:CONN_2
- Q1, Q10, Q13, Q2, Q5, Q6, Q9: symbol 2SC1815 -> juno-chorus-clone-rescue:2SC1815
- Q11, Q12, Q14, Q15, Q18, Q19, Q3, Q4, Q7, Q8: symbol 2SA1016 -> juno-chorus-clone-rescue:2SA1016
- Q16, Q17: symbol FET_N -> juno-chorus-clone-rescue:FET_N
- R1, R10, R11, R12, R13, R14, R15, R16, R17, R18, R19, R2, R20, R21, R22, R23, R24, R25, R26, R27, R28, R29, R3, R30, R31, R32, R33, R34, R35, R36, R37, R38, R39, R4, R40, R41, R42, R43, R44, R45, R46, R47, R48, R49, R5, R50, R51, R52, R53, R54, R55, R56, R57, R58, R59, R6, R60, R61, R62, R63, R64, R65, R66, R67, R68, R69, R7, R70, R71, R72, R73, R74, R75, R76, R77, R78, R79, R8, R80, R81, R82, R83, R84, R85, R86, R87, R88, R9: symbol R -> juno-chorus-clone-rescue:R
- RV1, RV2, RV3, RV4, RV5: symbol POT -> juno-chorus-clone-rescue:POT
- SW1: symbol SW_PUSH -> juno-chorus-clone-rescue:SW_PUSH
- U1, U10, U4, U9: symbol TL082 -> juno-chorus-clone-rescue:TL082
- U2: symbol LM7815CT -> juno-chorus-clone-rescue:LM7815CT
- U3: symbol LM7915CT -> juno-chorus-clone-rescue:LM7915CT
- U5, U6, U7, U8: symbol DIL8 -> juno-chorus-clone-rescue:DIL8
